File: minitel_interface.kicad_pcb (KiCad board)
At the start: 2 copper layers, 52.1 x 27.9 mm, 12 parts, among them U1 L7805, U2 MAX232

Commit message: Fix confusion on two pins on the MAX232
(original board requreid bodge wire)
Parts:
- added G***: LOGO, red_logo:RED_LOGO_7_6, F.Cu at (44.2, 37.6)
Connections:
- U2 pad 10: Net-(MinitelDIN5-Pad2) -> Net-(U2-Pad10)
- U2 pad 12: Net-(U2-Pad12) -> Net-(MinitelDIN5-Pad2)
Routing:
- net GND: track 52.3 -> 0.00 mm
- net REG_5V: track 36.2 -> 0.00 mm
- net Net-(MinitelDIN5-Pad2): track 32.4 -> 27.9 mm
- net Net-(C4-Pad2): track 4.35 -> 8.62 mm
- net Net-(PC-Serial1-Pad3): track 18.3 -> 21.4 mm
- net Net-(MinitelDIN5-Pad1): track 33.6 -> 34.3 mm
Other:
- board text added: "v2"
