File: minitel_interface.sch (KiCad schematic (older format))
At the start: 10 parts, among them U1 L7805, U2 MAX232

Commit message: Fix confusion on two pins on the MAX232
(original board requreid bodge wire)
Changed lines of the file:
@@
 EESchema Schematic File Version 4
+LIBS:minitel_interface-cache
 EELAYER 26 0
 EELAYER END
@@
 Wire Wire Line
 	2150 2500 2150 2750
-Wire Wire Line
-	2150 3800 4600 3800
 NoConn ~ 8900 3050
 NoConn ~ 8900 3250
@@
 NoConn ~ 6200 4200
 NoConn ~ 4600 4200
-NoConn ~ 4600 4000
 $Comp
 L power:+12V #PWR0105
@@
 Connection ~ 2150 2750
 Wire Wire Line
-	2150 2750 2150 3800
+	4600 4000 2150 4000
+Wire Wire Line
+	2150 2750 2150 4000
+NoConn ~ 4600 3800
 $EndSCHEMATC
